File: 0x708.kicad_pcb (KiCad board)
At the start: 2 copper layers, 381.5 x 173.1 mm, 261 parts, among them J1 USB_B, J2 AVR-ISP-6, SW1 Esc, SW10 F9, SW100 RWin, SW101 RCtrl, SW102 Left, SW103 Down, SW104 Right, SW105 Num0, SW106 Num., SW107 NumEnter2, SW108 LShift2, SW109 Backspace1, SW11 F10, SW110 ISOEnter, SW111 Num+1, SW112 LCtrl1.25, SW113 LWin1.25, SW114 LAlt1.25, SW115 Space6.25, SW116 NumEnter1, SW117 RESET, SW118 LCtrl1.5, SW119 LAlt1.5, SW12 F11, SW120 RAlt1.5, SW121 RCtrl1.5, SW122 Rotary_Encoder_Switch, SW13 F12, SW14 Ins, SW15 Home, SW16 PgUp, SW17 PrtSc, SW18 Del, SW19 End, SW2 F1, SW20 PgDn, SW21 ScrLk, SW22 `, SW23 1, SW24 2, SW25 3, SW26 4, SW27 5, SW28 6, SW29 7, SW3 F2, SW30 8, SW31 9, SW32 0, SW33 -, SW34 =, SW35 Backspace, SW36 Backspace2, SW37 NumLk, SW38 Num/, SW39 Num*, SW4 F3, SW40 Num-, SW41 Tab, SW42 Q, SW43 W, SW44 E, SW45 R, SW46 T, SW47 Y, SW48 U, SW49 I, SW5 F4, SW50 O, SW51 P, SW52 [, SW53 ], SW54 \, SW55 Num7, SW56 Num8, SW57 Num9, SW58 Num+, SW59 ALk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

Commit message: complete prototype
Parts:
- added H13: M2, MountingHole:MountingHole_2.2mm_M2, F.Cu at (148.6, 174.3)
- moved H8 185.9 mm to (210.5, 88.6)
- moved H12 149.0 mm to (353.4, 174.3)
- moved H3 122.3 mm to (148.6, 34.0), turned to 180 degrees
- moved H7 84.5 mm to (353.4, 88.6)
- moved H2 57.1 mm to (262.9, 34.0)
- moved H9 51.2 mm to (91.4, 88.6)
- moved H11 35.6 mm to (53.3, 136.2)
- moved H10 24.9 mm to (262.9, 136.2)
- renumbered H2 to H1, H12 to H10, H5 to H11, H14 to H12, H8 to H14, H7 to H15, H13 to H2, H11 to H3, H1 to H4, H4 to H5, H3 to H6, H10 to H7, H6 to H8
Routing:
- net COL6: track 413.4 -> 401.5 mm
